Commit message: bug fix in left hand xacro

File: src/allegro_hand_description/allegro_hand_description_left.xacro (robot description, xacro)
@@ -136,5 +136,5 @@
             </inertial>
         </link>
-        <joint name="joint_${finger_num*4+0}" type="revolute">
+        <joint name="joint_${finger_num*4+0}.0" type="revolute">
             <axis xyz="+1 0 0"/>
             <limit effort="15" velocity="7"
@@ -171,5 +171,5 @@
             </inertial>
         </link>
-        <joint name="joint_${finger_num*4+1}" type="revolute">
+        <joint name="joint_${finger_num*4+1}.0" type="revolute">
             <axis xyz="0 0 -1"/>
             <limit effort="15" velocity="7"
@@ -203,5 +203,5 @@
             </inertial>
         </link>
-        <joint name="joint_${finger_num*4+2}" type="revolute">
+        <joint name="joint_${finger_num*4+2}.0" type="revolute">
             <axis xyz="0 1 0"/>
             <limit effort="15" velocity="7"
@@ -236,5 +236,5 @@
             </inertial>
         </link>
-        <joint name="joint_${finger_num*4+3}" type="revolute">
+        <joint name="joint_${finger_num*4+3}.0" type="revolute">
             <axis xyz="0 1 0"/>
             <limit effort="15" velocity="7"
@@ -302,5 +302,5 @@
             </inertial>
         </link>
-        <joint name="joint_${finger_num*4+0}" type="revolute">
+        <joint name="joint_${finger_num*4+0}.0" type="revolute">
             <axis xyz="0 0 1"/>
             <limit effort="15" velocity="7"
@@ -335,5 +335,5 @@
             </inertial>
         </link>
-        <joint name="joint_${finger_num*4+1}" type="revolute">
+        <joint name="joint_${finger_num*4+1}.0" type="revolute">
             <limit effort="15" velocity="7"
                    lower="${limit_1_low+joint_safety_margin}"
@@ -367,5 +367,5 @@
             </inertial>
         </link>
-        <joint name="joint_${finger_num*4+2}" type="revolute">
+        <joint name="joint_${finger_num*4+2}.0" type="revolute">
             <axis xyz="0 1 0"/>
             <limit effort="15" velocity="7"
@@ -399,5 +399,5 @@
             </inertial>
         </link>
-        <joint name="joint_${finger_num*4+3}" type="revolute">
+        <joint name="joint_${finger_num*4+3}.0" type="revolute">
             <axis xyz="0 1 0"/>
             <limit effort="15" velocity="7"
